Commit message: fix: calibrate real lite_dummy link mass

File: robots/lite_dummy/urdf/lite.urdf (robot description, URDF)
Before this commit: robot lite, 20 links, 19 joints
Links:
- link left_hand: mass 0.153078 -> 0.161493
- link right_hand: mass 0.153078 -> 0.161493
- link right_shoulder_roll: mass 0.41 -> 0.41073
Joints:
- joint left_elbow_pitch: origin xyz=0.01 0 -0.08 rpy=-1.5708 0 -0 -> xyz=0.01 -0 -0.08 rpy=-1.5708 -0 -0
- joint left_shoulder_pitch: origin xyz=-0 0.09 0.39 rpy=-1.39626 0 0 -> xyz=0 0.09 0.39 rpy=-1.39626 -0 -0
- joint left_shoulder_roll: origin xyz=0 0 0 rpy=1.5708 0.174533 1.5708 -> xyz=0 0 -0 rpy=1.5708 0.174533 1.5708
- joint left_shoulder_yaw: origin xyz=-0 0.12 0 rpy=1.5708 -1.5708 0 -> xyz=0 0.12 -0 rpy=1.5708 -1.5708 0
- joint left_wrist_pitch: origin xyz=0 -0 0 rpy=0 1.5708 0 -> xyz=-0 0 0 rpy=0 1.5708 0
- joint left_wrist_yaw: origin xyz=-0.01 0.055 0 rpy=1.5708 0 0 -> xyz=-0.01 0.055 0 rpy=1.5708 -0 -0
- joint neck_pitch: origin xyz=-0 0.03 0 rpy=-0 1.5708 0 -> xyz=0 0.03 -0 rpy=0 1.5708 0
- joint neck_roll: origin xyz=0 0 0.03 rpy=1.5708 0 1.5708 -> xyz=0 -0 0.03 rpy=1.5708 0 1.5708
- joint neck_yaw: origin xyz=-0.01 -0 0.45 rpy=0 -0 0 -> xyz=-0.01 -0 0.45 rpy=0 -0 -0
- joint right_shoulder_pitch: origin xyz=0 -0.09 0.39 rpy=-1.74533 -0 -0 -> xyz=-0 -0.09 0.39 rpy=-1.74533 -0 -0
- joint right_shoulder_roll: origin xyz=-0 0 0 rpy=-1.5708 0.174533 -1.5708 -> xyz=0 0 0 rpy=-1.5708 0.174533 -1.5708
- joint right_shoulder_yaw: origin xyz=0 0.12 -0 rpy=1.5708 -1.5708 0 -> xyz=-0 0.12 -0 rpy=1.5708 -1.5708 0
- joint right_wrist_pitch: origin xyz=0 0 0 rpy=0 1.5708 0 -> xyz=-0 0 0 rpy=-0 1.5708 0
- joint right_wrist_roll: origin xyz=-0 0 -0.135 rpy=-1.5708 -0 0 -> xyz=0 0 -0.135 rpy=-1.5708 0 0
