Commit message: feat(lite_biped): re-export feet from CAD, model the full shoe sole
The shoe sat in the wrong place in the previous export. Re-exported from
Onshape (same document / configuration) offline via robot.pkl. The change is
confined to the two foot links: COM and visual origin move ~3.8 mm, inertia
rises 13-16%, mass unchanged. Standing height is NOT affected -- the sole plane
stays at exactly -0.775 m, so the training init pose, foot sites and every
height-dependent reward are untouched.

Foot colliders go from 2 boxes to 11 spheres per foot, now covering the whole
shoe bottom including the 21 mm toe upturn (y 58 -> 132 mm) that the boxes
never reached: only the flat patch was modelled before. Sphere centres sit on
the 3D lower convex hull of the sole -- the only points that can ever touch a
plane, since everything else is shadowed for every ground orientation -- and
are offset along the inward surface normal, so each is tangent to the shoe
rather than hovering above it (on a 25 deg toe facet those differ by 3.4 mm).

Validated by sweeping pitch -20..+40 deg x roll +-10 deg and comparing the
sphere set's lowest point against the real mesh at each pose: mean +0.46 mm,
max 2.07 mm. Standing support polygon 97.96 cm^2 across 8 load-bearing
spheres. Spheres are also cheaper than the boxes they replace -- box-plane
emits a contact per bottom corner, so grounded boxes cost up to 16 contacts
per foot versus 11 here, with no near-duplicate corner pairs to arbitrate.

Folded in from earlier work on this branch, because the regenerated artifacts
interleave it and splitting would mean committing a generator that disagrees
with its own output:

  - MJCF actuators switch from <motor> to <position>, putting the joint PD
    inside the physics step instead of sampling it once per controller_manager
    tick; regenerates lite_bimanual and lite_dummy too. Its unit test still
    asserted <motor> and was failing -- updated to match.
  - ankle_pitch four-bar linkage parameters in cad/ros2_control.json and the
    xacro generator.

uv run pytest: 1418 passed, 5 skipped.

Co-Authored-By: Claude Opus 5 (1M context) <noreply@anthropic.com>
Claude-Session: https://claude.ai/code/session_012QKJQ9hze1hMWXJpdPcjp3

File: robots/lite_biped/urdf/lite_biped.urdf (robot description, URDF)
Before this commit: robot lite_biped, 16 links, 15 joints
Links:
- link left_foot: geometry collision sphere radius=0.008; collision sphere radius=0.008
- link right_foot: geometry collision sphere radius=0.008; collision sphere radius=0.008
Joints:
- joint left_ankle_roll: origin xyz=-0 0.04 0 rpy=0 1.5708 0 -> xyz=0 0.04 -0 rpy=0 1.5708 0
- joint right_ankle_pitch: origin xyz=0.01 0 -0.34 rpy=-1.5708 0 0 -> xyz=0.01 0 -0.34 rpy=-1.5708 -0 -0
- joint right_ankle_roll: origin xyz=-0 0.04 -0 rpy=-0 1.5708 0 -> xyz=0 0.04 0 rpy=0 1.5708 0
- joint right_ankle_yaw: origin xyz=-0.015 0 -0 rpy=1.5708 -0 -0 -> xyz=-0.015 0 0 rpy=1.5708 -0 -0
- joint right_hip_yaw: origin xyz=-0 -0.0068404 -0.0187939 rpy=0 -1.22173 1.5708 -> xyz=-0 -0.0068404 -0.0187939 rpy=-0 -1.22173 1.5708

File: robots/lite_biped/xacro/lite_biped.description.xacro (robot description, xacro)
@@ -165,23 +165,77 @@
     <link name="left_foot">
       <inertial>
-        <origin xyz="0.00124938 0.0227876 0.0398042" rpy="0 0 0" />
+        <origin xyz="-0.00237479 0.023215 0.0359752" rpy="0 0 0" />
         <mass value="0.44" />
-        <inertia ixx="0.00133847" ixy="-3.31857e-06" ixz="-4.29633e-05" iyy="0.00119465" iyz="-0.000154848" izz="0.000481763" />
+        <inertia ixx="0.00151668" ixy="1.08029e-05" ixz="-4.76424e-05" iyy="0.00139101" iyz="-0.00016041" izz="0.000479544" />
       </inertial>
       <!-- Part left_foot_parts -->
       <collision>
-        <origin xyz="0 0.05 0.015" rpy="1.5708 0 0" />
-        <geometry>
-          <box size="0.065 0.12 0.03" />
-        </geometry>
-      </collision>
-      <collision>
-        <origin xyz="0 0.04 0.11" rpy="1.91986 0 0" />
-        <geometry>
-          <box size="0.07 0.05 0.03" />
-        </geometry>
-      </collision>
-      <visual>
-        <origin xyz="0.00124938 0.0227876 0.0398042" rpy="1.5708 -1.5708 0" />
+        <origin xyz="-0.0046 0.057 -0.05998" rpy="1.5708 0 0" />
+        <geometry>
+          <sphere radius="0.008" />
+        </geometry>
+      </collision>
+      <collision>
+        <origin xyz="-0.03941 0.057 -0.0259" rpy="1.5708 0 0" />
+        <geometry>
+          <sphere radius="0.008" />
+        </geometry>
+      </collision>
+      <collision>
+        <origin xyz="0.02804 0.057 -0.02442" rpy="1.5708 0 0" />
+        <geometry>
+          <sphere radius="0.008" />
+        </geometry>
+      </collision>
+      <collision>
+        <origin xyz="-0.04209 0.057 0.02764" rpy="1.5708 0 0" />
+        <geometry>
+          <sphere radius="0.008" />
+        </geometry>
+      </collision>
+      <collision>
+        <origin xyz="0.03476 0.057 0.02877" rpy="1.5708 0 0" />
+        <geometry>
+          <sphere radius="0.008" />
+        </geometry>
+      </collision>
+      <collision>
+        <origin xyz="-0.04432 0.057 0.0812" rpy="1.5708 0 0" />
+        <geometry>
+          <sphere radius="0.008" />
+        </geometry>
+      </collision>
+      <collision>
+        <origin xyz="0.04148 0.057 0.08196" rpy="1.5708 0 0" />
+        <geometry>
+          <sphere radius="0.008" />
+        </geometry>
+      </collision>
+      <collision>
+        <origin xyz="-0.00047 0.057 0.09173" rpy="1.5708 0 0" />
+        <geometry>
+          <sphere radius="0.008" />
+        </geometry>
+      </collision>
+      <collision>
+        <origin xyz="-0.03438 0.04891 0.12489" rpy="1.5708 0 0" />
+        <geometry>
+          <sphere radius="0.008" />
+        </geometry>
+      </collision>
+      <collision>
+        <origin xyz="0.03932 0.04853 0.12597" rpy="1.5708 0 0" />
+        <geometry>
+          <sphere radius="0.008" />
+        </geometry>
+      </collision>
+      <collision>
+        <origin xyz="0.00465 0.03713 0.14874" rpy="1.5708 0 0" />
+        <geometry>
+          <sphere radius="0.008" />
+        </geometry>
+      </collision>
+      <visual>
+        <origin xyz="-0.00237479 0.023215 0.0359752" rpy="1.5708 -1.5708 0" />
         <geometry>
           <mesh filename="${mesh_root}/left_foot_visual.stl" />
@@ -194,5 +248,5 @@
     <!-- Joint from left_ankle_pitch to left_foot -->
     <joint name="left_ankle_roll" type="revolute">
-      <origin xyz="-0 0.04 0" rpy="0 1.5708 0" />
+      <origin xyz="0 0.04 -0" rpy="0 1.5708 0" />
       <parent link="left_ankle_pitch" />
       <child link="left_foot" />
@@ -276,5 +330,5 @@
     <link name="right_hip_roll">
       <inertial>
-        <origin xyz="-1.13349e-07 0.0525083 -0.0652488" rpy="0 0 0" />
+        <origin xyz="2.6715e-08 0.0525085 -0.0652483" rpy="0 0 0" />
         <mass value="0.93" />
         <inertia ixx="0.00263147" ixy="2.71e-10" ixz="6.079e-09" iyy="0.00142387" iyz="-0.000651423" izz="0.00255493" />
@@ -282,5 +336,5 @@
       <!-- Part right_hip_roll_parts -->
       <collision>
-        <origin xyz="-0 0.181098 -0.0871979" rpy="1.22173 0 0" />
+        <origin xyz="1.40064e-07 0.181098 -0.0871974" rpy="1.22173 0 -0" />
         <geometry>
           <cylinder length="0.15" radius="0.05" />
@@ -288,5 +342,5 @@
       </collision>
       <visual>
-        <origin xyz="-1.13349e-07 0.0525083 -0.0652488" rpy="0 -1.22173 1.5708" />
+        <origin xyz="2.6715e-08 0.0525085 -0.0652483" rpy="0 -1.22173 1.5708" />
         <geometry>
           <mesh filename="${mesh_root}/right_hip_roll_visual.stl" />
@@ -306,5 +360,5 @@
       <!-- Part right_hip_yaw_parts -->
       <visual>
-        <origin xyz="0.00130421 2.35733e-05 -0.237299" rpy="0 0 0" />
+        <origin xyz="0.00130421 2.35733e-05 -0.237299" rpy="0 0 -0" />
         <geometry>
           <mesh filename="${mesh_root}/right_hip_yaw_visual.stl" />
@@ -330,5 +384,5 @@
       </collision>
       <visual>
-        <origin xyz="-0.0048642 0.0372186 0.000224747" rpy="1.5708 -0 0" />
+        <origin xyz="-0.0048642 0.0372186 0.000224747" rpy="1.5708 0 0" />
         <geometry>
           <mesh filename="${mesh_root}/right_knee_pitch_visual.stl" />
@@ -348,5 +402,5 @@
       <!-- Part right_ankle_yaw_parts -->
       <visual>
-        <origin xyz="-0.00304908 -0.0015054 -0.185348" rpy="0 0 0" />
+        <origin xyz="-0.00304908 -0.0015054 -0.185348" rpy="0 0 -0" />
         <geometry>
           <mesh filename="${mesh_root}/right_ankle_yaw_visual.stl" />
@@ -366,5 +420,5 @@
       <!-- Part right_ankle_pitch_parts -->
       <visual>
-        <origin xyz="-0.00384209 0.0297371 3.1396e-08" rpy="1.5708 -0 0" />
+        <origin xyz="-0.00384209 0.0297371 3.1396e-08" rpy="1.5708 0 0" />
         <geometry>
           <mesh filename="${mesh_root}/right_ankle_pitch_visual.stl" />
@@ -378,23 +432,77 @@
     <link name="right_foot">
       <inertial>
-        <origin xyz="-0.0012494 0.0227876 0.039804" rpy="0 0 0" />
+        <origin xyz="0.0023746 0.0232151 0.0359757" rpy="0 0 0" />
         <mass value="0.44" />
-        <inertia ixx="0.00133847" ixy="3.3182e-06" ixz="4.29635e-05" iyy="0.00119465" iyz="-0.000154847" izz="0.000481763" />
+        <inertia ixx="0.00151669" ixy="-1.0799e-05" ixz="4.76345e-05" iyy="0.00139101" iyz="-0.000160415" izz="0.000479546" />
       </inertial>
       <!-- Part right_foot_parts -->
       <collision>
-        <origin xyz="0 0.05 0.015" rpy="1.5708 0 -0" />
-        <geometry>
-          <box size="0.065 0.12 0.03" />
-        </geometry>
-      </collision>
-      <collision>
-        <origin xyz="0 0.04 0.11" rpy="1.91986 0 -0" />
-        <geometry>
-          <box size="0.07 0.05 0.03" />
-        </geometry>
-      </collision>
-      <visual>
-        <origin xyz="-0.0012494 0.0227876 0.039804" rpy="1.5708 -1.5708 0" />
+        <origin xyz="0.0046 0.057 -0.05998" rpy="1.5708 0 0" />
+        <geometry>
+          <sphere radius="0.008" />
+        </geometry>
+      </collision>
+      <collision>
+        <origin xyz="0.03941 0.057 -0.0259" rpy="1.5708 0 0" />
+        <geometry>
+          <sphere radius="0.008" />
+        </geometry>
+      </collision>
+      <collision>
+        <origin xyz="-0.02804 0.057 -0.02442" rpy="1.5708 0 0" />
+        <geometry>
+          <sphere radius="0.008" />
+        </geometry>
+      </collision>
+      <collision>
+        <origin xyz="0.04209 0.057 0.02764" rpy="1.5708 0 0" />
+        <geometry>
+          <sphere radius="0.008" />
+        </geometry>
+      </collision>
+      <collision>
+        <origin xyz="-0.03476 0.057 0.02877" rpy="1.5708 0 0" />
+        <geometry>
+          <sphere radius="0.008" />
+        </geometry>
+      </collision>
+      <collision>
+        <origin xyz="0.04432 0.057 0.0812" rpy="1.5708 0 0" />
+        <geometry>
+          <sphere radius="0.008" />
+        </geometry>
+      </collision>
+      <collision>
+        <origin xyz="-0.04148 0.057 0.08196" rpy="1.5708 0 0" />
+        <geometry>
+          <sphere radius="0.008" />
+        </geometry>
+      </collision>
+      <collision>
+        <origin xyz="0.00047 0.057 0.09173" rpy="1.5708 0 0" />
+        <geometry>
+          <sphere radius="0.008" />
+        </geometry>
+      </collision>
+      <collision>
+        <origin xyz="0.03438 0.04891 0.12489" rpy="1.5708 0 0" />
+        <geometry>
+          <sphere radius="0.008" />
+        </geometry>
+      </collision>
+      <collision>
+        <origin xyz="-0.03932 0.04853 0.12597" rpy="1.5708 0 0" />
+        <geometry>
+          <sphere radius="0.008" />
+        </geometry>
+      </collision>
+      <collision>
+        <origin xyz="-0.00465 0.03713 0.14874" rpy="1.5708 0 0" />
+        <geometry>
+          <sphere radius="0.008" />
+        </geometry>
+      </collision>
+      <visual>
+        <origin xyz="0.0023746 0.0232151 0.0359757" rpy="1.5708 -1.5708 0" />
         <geometry>
           <mesh filename="${mesh_root}/right_foot_visual.stl" />
@@ -407,5 +515,5 @@
     <!-- Joint from right_ankle_pitch to right_foot -->
     <joint name="right_ankle_roll" type="revolute">
-      <origin xyz="-0 0.04 -0" rpy="-0 1.5708 0" />
+      <origin xyz="0 0.04 0" rpy="0 1.5708 0" />
       <parent link="right_ankle_pitch" />
       <child link="right_foot" />
@@ -416,5 +524,5 @@
     <!-- Joint from right_ankle_yaw to right_ankle_pitch -->
     <joint name="right_ankle_pitch" type="revolute">
-      <origin xyz="0.01 0 -0.34" rpy="-1.5708 0 0" />
+      <origin xyz="0.01 0 -0.34" rpy="-1.5708 -0 -0" />
       <parent link="right_ankle_yaw" />
       <child link="right_ankle_pitch" />
@@ -425,5 +533,5 @@
     <!-- Joint from right_knee_pitch to right_ankle_yaw -->
     <joint name="right_ankle_yaw" type="revolute">
-      <origin xyz="-0.015 0 -0" rpy="1.5708 -0 -0" />
+      <origin xyz="-0.015 0 0" rpy="1.5708 -0 -0" />
       <parent link="right_knee_pitch" />
       <child link="right_ankle_yaw" />
@@ -443,5 +551,5 @@
     <!-- Joint from right_hip_roll to right_hip_yaw -->
     <joint name="right_hip_yaw" type="revolute">
-      <origin xyz="-0 -0.0068404 -0.0187939" rpy="0 -1.22173 1.5708" />
+      <origin xyz="-0 -0.0068404 -0.0187939" rpy="-0 -1.22173 1.5708" />
       <parent link="right_hip_roll" />
       <child link="right_hip_yaw" />

File: robots/lite_biped/xacro/lite_biped.ros2_control.xacro (robot description, xacro)
@@ -7,5 +7,8 @@
                params="name can_id model direction
                        lower_limit upper_limit torque_limit current_limit
-                       use_fake_hardware use_sim">
+                       use_fake_hardware use_sim
+                       use_linkage:=true linkage_ground:=0
+                       linkage_crank_in:=0 linkage_coupler:=0 linkage_crank_out:=0
+                       linkage_alpha_zero:=0 linkage_sign:=1">
     <joint name="${name}">
       <command_interface name="position"/>
@@ -25,8 +28,27 @@
         <param name="torque_limit">${torque_limit}</param>
         <param name="current_limit">${current_limit}</param>
+        <!-- Four-bar transmission geometry, for joints that declare one in
+             ros2_control.json. The geometry is a PHYSICAL FACT so it is always
+             published: calibrate_robot reads it from /robot_description to refer
+             the URDF joint limits into actuator space, even on the runs where the
+             hardware plugin must NOT apply the transform. `linkage_enabled`
+             (= the use_linkage arg) is what switches the plugin's behaviour:
+             false during calibration, which needs raw actuator angles. With it
+             true, RobstrideSystem converts joint<->actuator through the linkage
+             and refers the commanded impedance by J^2, so /joint_states and every
+             controller speak true joint space. -->
+        <xacro:if value="${linkage_ground > 0}">
+          <param name="linkage_ground">${linkage_ground}</param>
+          <param name="linkage_crank_in">${linkage_crank_in}</param>
+          <param name="linkage_coupler">${linkage_coupler}</param>
+          <param name="linkage_crank_out">${linkage_crank_out}</param>
+          <param name="linkage_alpha_zero">${linkage_alpha_zero}</param>
+          <param name="linkage_sign">${linkage_sign}</param>
+          <param name="linkage_enabled">${use_linkage}</param>
+        </xacro:if>
       </xacro:unless>
     </joint>
   </xacro:macro>
-  <xacro:macro name="lite_biped_left_leg_joints" params="use_fake_hardware use_sim">
+  <xacro:macro name="lite_biped_left_leg_joints" params="use_fake_hardware use_sim use_linkage:=true">
     <xacro:lite_biped_joint name="left_hip_pitch" can_id="31" model="rs-06" direction="-1"
                       lower_limit="-2.35619" upper_limit="0.785398"
@@ -52,5 +74,9 @@
                       lower_limit="-0.523599" upper_limit="0.872665"
                       torque_limit="14.0" current_limit="16"
-                      use_fake_hardware="${use_fake_hardware}" use_sim="${use_sim}"/>
+                      use_fake_hardware="${use_fake_hardware}" use_sim="${use_sim}"
+                      linkage_ground="160.449369" linkage_crank_in="40.0"
+                      linkage_coupler="150.0" linkage_crank_out="40.0"
+                      linkage_alpha_zero="338.82213" linkage_sign="1"
+                      use_linkage="${use_linkage}"/>
     <xacro:lite_biped_joint name="left_ankle_roll" can_id="37" model="rs-05" direction="-1"
                       lower_limit="-0.349066" upper_limit="0.349066"
@@ -58,5 +84,5 @@
                       use_fake_hardware="${use_fake_hardware}" use_sim="${use_sim}"/>
   </xacro:macro>
-  <xacro:macro name="lite_biped_right_leg_joints" params="use_fake_hardware use_sim">
+  <xacro:macro name="lite_biped_right_leg_joints" params="use_fake_hardware use_sim use_linkage:=true">
     <xacro:lite_biped_joint name="right_hip_pitch" can_id="41" model="rs-06" direction="1"
                       lower_limit="-2.35619" upper_limit="0.785398"
@@ -82,5 +108,9 @@
                       lower_limit="-0.523599" upper_limit="0.872665"
                       torque_limit="14.0" current_limit="16"
-                      use_fake_hardware="${use_fake_hardware}" use_sim="${use_sim}"/>
+                      use_fake_hardware="${use_fake_hardware}" use_sim="${use_sim}"
+                      linkage_ground="160.449369" linkage_crank_in="40.0"
+                      linkage_coupler="150.0" linkage_crank_out="40.0"
+                      linkage_alpha_zero="338.82213" linkage_sign="1"
+                      use_linkage="${use_linkage}"/>
     <xacro:lite_biped_joint name="right_ankle_roll" can_id="47" model="rs-05" direction="-1"
                       lower_limit="-0.349066" upper_limit="0.349066"
@@ -121,5 +151,5 @@
        single flat joint list to controllers. -->
   <xacro:macro name="lite_biped_ros2_control_real"
-               params="mode can_interface_left can_interface_right calibration_file imu_port">
+               params="mode can_interface_left can_interface_right calibration_file imu_port use_linkage">
     <ros2_control name="LiteBipedLeftLeg" type="system">
       <hardware>
@@ -128,5 +158,5 @@
         <param name="calibration_file">${calibration_file}</param>
       </hardware>
-      <xacro:lite_biped_left_leg_joints use_fake_hardware="false" use_sim="false"/>
+      <xacro:lite_biped_left_leg_joints use_fake_hardware="false" use_sim="false" use_linkage="${use_linkage}"/>
     </ros2_control>
     <ros2_control name="LiteBipedRightLeg" type="system">
@@ -136,5 +166,5 @@
         <param name="calibration_file">${calibration_file}</param>
       </hardware>
-      <xacro:lite_biped_right_leg_joints use_fake_hardware="false" use_sim="false"/>
+      <xacro:lite_biped_right_leg_joints use_fake_hardware="false" use_sim="false" use_linkage="${use_linkage}"/>
     </ros2_control>
     <ros2_control name="LiteBipedIMU" type="sensor">
@@ -161,5 +191,5 @@
   <xacro:macro name="lite_biped_ros2_control"
                params="name use_fake_hardware use_sim mode
-                       can_interface_left can_interface_right calibration_file imu_port">
+                       can_interface_left can_interface_right calibration_file imu_port use_linkage">
     <xacro:if value="${use_sim or use_fake_hardware}">
       <xacro:lite_biped_ros2_control_combined name="${name}"
@@ -171,5 +201,6 @@
         can_interface_right="${can_interface_right}"
         calibration_file="${calibration_file}"
-        imu_port="${imu_port}"/>
+        imu_port="${imu_port}"
+        use_linkage="${use_linkage}"/>
     </xacro:unless>
   </xacro:macro>

File: robots/lite_biped/xacro/lite_biped.urdf.xacro (robot description, xacro)
@@ -9,4 +9,5 @@
   <xacro:arg name="calibration_file" default=""/>
   <xacro:arg name="imu_port" default="/dev/ttyUSB0"/>
+  <xacro:arg name="use_linkage" default="true"/>
   <xacro:include filename="$(find lite_description)/robots/lite_biped/xacro/lite_biped.description.xacro"/>
   <xacro:include filename="$(find lite_description)/robots/lite_biped/xacro/lite_biped.ros2_control.xacro"/>
@@ -20,4 +21,5 @@
     can_interface_right="$(arg can_interface_right)"
     calibration_file="$(arg calibration_file)"
-    imu_port="$(arg imu_port)"/>
+    imu_port="$(arg imu_port)"
+    use_linkage="$(arg use_linkage)"/>
 </robot>
