Commit message: Name the sim and mock components as the real ones, and declare their safety gpio
The mock and MuJoCo backends collapsed every bus into one component, so a robot
was LiteHardware in simulation and LiteLeftArm + LiteRightArm on hardware.
Anything keyed by component name therefore meant a different thing per backend:
a controller's safety_components, the hardware_spawner, the manager's
hardware_components_initial_state. The practical cost was that
SafetyMonitorController, which names the real components, could not load in
simulation at all -- the one place the fault-handover path can be exercised
without a robot.

The combined macro now emits one block per bus with the real backend's own
block_name. Nothing in the vendored mujoco_ros2_control needs changing: it
already iterates every <ros2_control> block and imports each one.

Mock also gains a <gpio> per component carrying safety_level and safety_flags.
The real drivers export those from
export_unlisted_state_interface_descriptions(), which mock_components has no
equivalent for; the base class parses gpio state interfaces straight from the
description (hardware_component_interface.cpp:163) and GenericSystem does not
override that path, so declaring them is enough. MuJoCo is deliberately left
out: our MujocoSystem overrides the deprecated by-value
export_state_interfaces(), which bypasses the base class's gpio handling, so a
gpio there would promise interfaces that never appear.

An IMU with a real component gets a matching sensor block in sim. A sim-only one
has no name to match and stays nested, which is what
test_imu_without_real_plugin_emits_no_sensor_component pins.

combined_block_name is deleted from every cad/ros2_control.json: with the real
names in use it is read by nothing.

Two tests lock this in -- component names equal across sim and real, mock a
subset since it cannot back an IMU, and every mock system block carrying both
safety interfaces. Both were negative-controlled against the committed
artifacts, since that is what they read.

Co-Authored-By: Claude Opus 5 (1M context) <noreply@anthropic.com>
Claude-Session: https://claude.ai/code/session_01EotyWG9YmYvg5xE2v3Zkpt

File: robots/lite_bimanual/xacro/lite_bimanual.ros2_control.xacro (robot description, xacro)
@@ -72,7 +72,10 @@
                                current_limit="14"/>
   </xacro:macro>
-  <!-- Combined single block for the mock and MuJoCo backends. -->
-  <xacro:macro name="lite_bimanual_ros2_control_combined" params="name sim_mujoco">
-    <ros2_control name="${name}" type="system">
+  <!-- Mock and MuJoCo backends. One block per bus, carrying the same component
+       names as the real backend, so anything keyed by component name means the
+       same thing on every backend: a controller's safety_components, the
+       hardware_spawner, the manager's hardware_components_initial_state. -->
+  <xacro:macro name="lite_bimanual_ros2_control_combined" params="sim_mujoco">
+    <ros2_control name="LiteLeftArm" type="system">
       <hardware>
         <xacro:if value="${sim_mujoco}">
@@ -84,5 +87,27 @@
       </hardware>
       <xacro:lite_bimanual_left_arm_joints/>
+      <xacro:unless value="${sim_mujoco}">
+        <gpio name="LiteLeftArm">
+          <state_interface name="safety_level"/>
+          <state_interface name="safety_flags"/>
+        </gpio>
+      </xacro:unless>
+    </ros2_control>
+    <ros2_control name="LiteRightArm" type="system">
+      <hardware>
+        <xacro:if value="${sim_mujoco}">
+          <plugin>mujoco_ros2_control/MujocoSystem</plugin>
+        </xacro:if>
+        <xacro:unless value="${sim_mujoco}">
+          <plugin>mock_components/GenericSystem</plugin>
+        </xacro:unless>
+      </hardware>
       <xacro:lite_bimanual_right_arm_joints/>
+      <xacro:unless value="${sim_mujoco}">
+        <gpio name="LiteRightArm">
+          <state_interface name="safety_level"/>
+          <state_interface name="safety_flags"/>
+        </gpio>
+      </xacro:unless>
     </ros2_control>
   </xacro:macro>
@@ -112,8 +137,8 @@
        sim_mujoco wins over use_mock_hardware. -->
   <xacro:macro name="lite_bimanual_ros2_control"
-               params="name use_mock_hardware sim_mujoco can_interface_left can_interface_right
+               params="use_mock_hardware sim_mujoco can_interface_left can_interface_right
                        calibration_file">
     <xacro:if value="${sim_mujoco or use_mock_hardware}">
-      <xacro:lite_bimanual_ros2_control_combined name="${name}" sim_mujoco="${sim_mujoco}"/>
+      <xacro:lite_bimanual_ros2_control_combined sim_mujoco="${sim_mujoco}"/>
     </xacro:if>
     <xacro:unless value="${sim_mujoco or use_mock_hardware}">

File: robots/lite_bimanual/xacro/lite_bimanual.urdf.xacro (robot description, xacro)
@@ -11,5 +11,4 @@
   <xacro:lite_bimanual_description/>
   <xacro:lite_bimanual_ros2_control
-    name="LiteHardware"
     use_mock_hardware="$(arg use_mock_hardware)"
     sim_mujoco="$(arg sim_mujoco)"

File: robots/lite_biped/xacro/lite_biped.ros2_control.xacro (robot description, xacro)
@@ -117,7 +117,10 @@
                             current_limit="14"/>
   </xacro:macro>
-  <!-- Combined single block for the mock and MuJoCo backends. -->
-  <xacro:macro name="lite_biped_ros2_control_combined" params="name sim_mujoco">
-    <ros2_control name="${name}" type="system">
+  <!-- Mock and MuJoCo backends. One block per bus, carrying the same component
+       names as the real backend, so anything keyed by component name means the
+       same thing on every backend: a controller's safety_components, the
+       hardware_spawner, the manager's hardware_components_initial_state. -->
+  <xacro:macro name="lite_biped_ros2_control_combined" params="sim_mujoco">
+    <ros2_control name="LiteBipedLeftLeg" type="system">
       <hardware>
         <xacro:if value="${sim_mujoco}">
@@ -129,6 +132,33 @@
       </hardware>
       <xacro:lite_biped_left_leg_joints/>
+      <xacro:unless value="${sim_mujoco}">
+        <gpio name="LiteBipedLeftLeg">
+          <state_interface name="safety_level"/>
+          <state_interface name="safety_flags"/>
+        </gpio>
+      </xacro:unless>
+    </ros2_control>
+    <ros2_control name="LiteBipedRightLeg" type="system">
+      <hardware>
+        <xacro:if value="${sim_mujoco}">
+          <plugin>mujoco_ros2_control/MujocoSystem</plugin>
+        </xacro:if>
+        <xacro:unless value="${sim_mujoco}">
+          <plugin>mock_components/GenericSystem</plugin>
+        </xacro:unless>
+      </hardware>
       <xacro:lite_biped_right_leg_joints/>
-      <xacro:if value="${sim_mujoco}">
+      <xacro:unless value="${sim_mujoco}">
+        <gpio name="LiteBipedRightLeg">
+          <state_interface name="safety_level"/>
+          <state_interface name="safety_flags"/>
+        </gpio>
+      </xacro:unless>
+    </ros2_control>
+    <xacro:if value="${sim_mujoco}">
+      <ros2_control name="LiteBipedIMU" type="sensor">
+        <hardware>
+          <plugin>mujoco_ros2_control/MujocoSystem</plugin>
+        </hardware>
         <sensor name="base_imu">
           <state_interface name="orientation.x"/>
@@ -143,6 +173,6 @@
           <state_interface name="linear_acceleration.z"/>
         </sensor>
-      </xacro:if>
-    </ros2_control>
+      </ros2_control>
+    </xacro:if>
   </xacro:macro>
   <!-- Real hardware: one <ros2_control> block per CAN bus. The controller_manager
@@ -190,8 +220,8 @@
        sim_mujoco wins over use_mock_hardware. -->
   <xacro:macro name="lite_biped_ros2_control"
-               params="name use_mock_hardware sim_mujoco can_interface_left can_interface_right
+               params="use_mock_hardware sim_mujoco can_interface_left can_interface_right
                        calibration_file imu_port use_linkage">
     <xacro:if value="${sim_mujoco or use_mock_hardware}">
-      <xacro:lite_biped_ros2_control_combined name="${name}" sim_mujoco="${sim_mujoco}"/>
+      <xacro:lite_biped_ros2_control_combined sim_mujoco="${sim_mujoco}"/>
     </xacro:if>
     <xacro:unless value="${sim_mujoco or use_mock_hardware}">

File: robots/lite_biped/xacro/lite_biped.urdf.xacro (robot description, xacro)
@@ -13,5 +13,4 @@
   <xacro:lite_biped_description/>
   <xacro:lite_biped_ros2_control
-    name="LiteBipedHardware"
     use_mock_hardware="$(arg use_mock_hardware)"
     sim_mujoco="$(arg sim_mujoco)"

File: robots/lite_biped_debug/xacro/lite_biped_debug.ros2_control.xacro (robot description, xacro)
@@ -117,7 +117,10 @@
                                   torque_limit="5.5" current_limit="14"/>
   </xacro:macro>
-  <!-- Combined single block for the mock and MuJoCo backends. -->
-  <xacro:macro name="lite_biped_debug_ros2_control_combined" params="name sim_mujoco">
-    <ros2_control name="${name}" type="system">
+  <!-- Mock and MuJoCo backends. One block per bus, carrying the same component
+       names as the real backend, so anything keyed by component name means the
+       same thing on every backend: a controller's safety_components, the
+       hardware_spawner, the manager's hardware_components_initial_state. -->
+  <xacro:macro name="lite_biped_debug_ros2_control_combined" params="sim_mujoco">
+    <ros2_control name="LiteBipedLeftLeg" type="system">
       <hardware>
         <xacro:if value="${sim_mujoco}">
@@ -129,6 +132,33 @@
       </hardware>
       <xacro:lite_biped_debug_left_leg_joints/>
+      <xacro:unless value="${sim_mujoco}">
+        <gpio name="LiteBipedLeftLeg">
+          <state_interface name="safety_level"/>
+          <state_interface name="safety_flags"/>
+        </gpio>
+      </xacro:unless>
+    </ros2_control>
+    <ros2_control name="LiteBipedRightLeg" type="system">
+      <hardware>
+        <xacro:if value="${sim_mujoco}">
+          <plugin>mujoco_ros2_control/MujocoSystem</plugin>
+        </xacro:if>
+        <xacro:unless value="${sim_mujoco}">
+          <plugin>mock_components/GenericSystem</plugin>
+        </xacro:unless>
+      </hardware>
       <xacro:lite_biped_debug_right_leg_joints/>
-      <xacro:if value="${sim_mujoco}">
+      <xacro:unless value="${sim_mujoco}">
+        <gpio name="LiteBipedRightLeg">
+          <state_interface name="safety_level"/>
+          <state_interface name="safety_flags"/>
+        </gpio>
+      </xacro:unless>
+    </ros2_control>
+    <xacro:if value="${sim_mujoco}">
+      <ros2_control name="LiteBipedIMU" type="sensor">
+        <hardware>
+          <plugin>mujoco_ros2_control/MujocoSystem</plugin>
+        </hardware>
         <sensor name="base_imu">
           <state_interface name="orientation.x"/>
@@ -143,6 +173,6 @@
           <state_interface name="linear_acceleration.z"/>
         </sensor>
-      </xacro:if>
-    </ros2_control>
+      </ros2_control>
+    </xacro:if>
   </xacro:macro>
   <!-- Real hardware: one <ros2_control> block per CAN bus. The controller_manager
@@ -190,8 +220,8 @@
        sim_mujoco wins over use_mock_hardware. -->
   <xacro:macro name="lite_biped_debug_ros2_control"
-               params="name use_mock_hardware sim_mujoco can_interface_left can_interface_right
+               params="use_mock_hardware sim_mujoco can_interface_left can_interface_right
                        calibration_file imu_port use_linkage">
     <xacro:if value="${sim_mujoco or use_mock_hardware}">
-      <xacro:lite_biped_debug_ros2_control_combined name="${name}" sim_mujoco="${sim_mujoco}"/>
+      <xacro:lite_biped_debug_ros2_control_combined sim_mujoco="${sim_mujoco}"/>
     </xacro:if>
     <xacro:unless value="${sim_mujoco or use_mock_hardware}">

File: robots/lite_biped_debug/xacro/lite_biped_debug.urdf.xacro (robot description, xacro)
@@ -13,5 +13,4 @@
   <xacro:lite_biped_debug_description/>
   <xacro:lite_biped_debug_ros2_control
-    name="LiteBipedHardware"
     use_mock_hardware="$(arg use_mock_hardware)"
     sim_mujoco="$(arg sim_mujoco)"

File: robots/lite_dummy/xacro/lite_dummy.ros2_control.xacro (robot description, xacro)
@@ -72,7 +72,10 @@
                             current_limit="14"/>
   </xacro:macro>
-  <!-- Combined single block for the mock and MuJoCo backends. -->
-  <xacro:macro name="lite_dummy_ros2_control_combined" params="name sim_mujoco">
-    <ros2_control name="${name}" type="system">
+  <!-- Mock and MuJoCo backends. One block per bus, carrying the same component
+       names as the real backend, so anything keyed by component name means the
+       same thing on every backend: a controller's safety_components, the
+       hardware_spawner, the manager's hardware_components_initial_state. -->
+  <xacro:macro name="lite_dummy_ros2_control_combined" params="sim_mujoco">
+    <ros2_control name="LiteLeftArm" type="system">
       <hardware>
         <xacro:if value="${sim_mujoco}">
@@ -84,5 +87,27 @@
       </hardware>
       <xacro:lite_dummy_left_arm_joints/>
+      <xacro:unless value="${sim_mujoco}">
+        <gpio name="LiteLeftArm">
+          <state_interface name="safety_level"/>
+          <state_interface name="safety_flags"/>
+        </gpio>
+      </xacro:unless>
+    </ros2_control>
+    <ros2_control name="LiteRightArm" type="system">
+      <hardware>
+        <xacro:if value="${sim_mujoco}">
+          <plugin>mujoco_ros2_control/MujocoSystem</plugin>
+        </xacro:if>
+        <xacro:unless value="${sim_mujoco}">
+          <plugin>mock_components/GenericSystem</plugin>
+        </xacro:unless>
+      </hardware>
       <xacro:lite_dummy_right_arm_joints/>
+      <xacro:unless value="${sim_mujoco}">
+        <gpio name="LiteRightArm">
+          <state_interface name="safety_level"/>
+          <state_interface name="safety_flags"/>
+        </gpio>
+      </xacro:unless>
     </ros2_control>
   </xacro:macro>
@@ -112,8 +137,8 @@
        sim_mujoco wins over use_mock_hardware. -->
   <xacro:macro name="lite_dummy_ros2_control"
-               params="name use_mock_hardware sim_mujoco can_interface_left can_interface_right
+               params="use_mock_hardware sim_mujoco can_interface_left can_interface_right
                        calibration_file">
     <xacro:if value="${sim_mujoco or use_mock_hardware}">
-      <xacro:lite_dummy_ros2_control_combined name="${name}" sim_mujoco="${sim_mujoco}"/>
+      <xacro:lite_dummy_ros2_control_combined sim_mujoco="${sim_mujoco}"/>
     </xacro:if>
     <xacro:unless value="${sim_mujoco or use_mock_hardware}">

File: robots/lite_dummy/xacro/lite_dummy.urdf.xacro (robot description, xacro)
@@ -11,5 +11,4 @@
   <xacro:lite_dummy_description/>
   <xacro:lite_dummy_ros2_control
-    name="LiteHardware"
     use_mock_hardware="$(arg use_mock_hardware)"
     sim_mujoco="$(arg sim_mujoco)"
